Commit message: Update four jackal, six jackal navigation

File: src/jackal/jackal_description_rtab/urdf/multi_jackal.urdf.xacro (robot description, xacro)
@@ -235,60 +235,43 @@
     <origin xyz="${mount_spacing} 0 0" />
   </joint>
-    <!-- zed camera -->
-  <link name="zed_camera_link">
+  <!-- stereo camera -->
+  <joint name="left_camera_joint" type="fixed">
+    <origin xyz="0.7 0 0.3" rpy="0 0 0"/>
+    <parent link="base_link"/>
+    <child link="left_camera_link"/>
+  </joint>
+  <link name="left_camera_link">
+    <visual>
+      <geometry>
+        <box size="0.02 0.02 0.02"/>
+      </geometry>
+      <material name="blue"/>
+    </visual>
+    <collision>
+      <geometry>
+        <box size="0.02 0.02 0.02"/>
+      </geometry>
+    </collision>
     <inertial>
-      <mass value="1e-5" />
-      <origin xyz="0 0 0" rpy="0 0 0"/>
-      <inertia ixx="1e-6" ixy="0" ixz="0" iyy="1e-6" iyz="0" izz="1e-6" />
+      <origin xyz="0 0 1" rpy="0 0 0"/>
+      <mass value="0.0"/>
+      <inertia
+        ixx="1.0" ixy="0.0" ixz="0.0"
+        iyy="1.0" iyz="0.0"
+        izz="1.0"/>
     </inertial>
-    <collision>
-      <origin xyz="0 0 0" rpy="0 0 0"/>
-      <geometry>
-        <box size="0.033 0.175 0.030"/>
-      </geometry>
-    </collision>
-    <visual>
-      <origin xyz="0 0 0" rpy="0 0 0"/>
-      <geometry>
-        <box size="0.033 0.175 0.030"/>
-      </geometry>
-      <material name="red"/>
-    </visual>
-  </link>
-  <joint name="zed_camera_joint" type="fixed">
-    <origin xyz="0.390 0 0.04" rpy="0 0 0"/>
-    <parent link="chassis_link"/>
-    <child link="zed_camera_link"/>
-    <axis xyz="0 0 1" />
-    <!-- <limit lower="0.0" upper="0.0" effort="0.0" velocity="0.0" /> -->
-  </joint>
-  <!-- zed camera lenses -->
-  <!-- It seems these have to have a non-zero mass to have a camera attached? -->
-  <link name="camera_link"><!-- this needs to match the name in zed_wrapper/zed_tf.launch -->
-    <inertial>
-      <mass value="1e-5" />
-      <origin xyz="0 0 0" rpy="0 0 0"/>
-      <inertia ixx="1e-6" ixy="0" ixz="0" iyy="1e-6" iyz="0" izz="1e-6" />
-    </inertial>
-  </link>
-  <link name="zed_camera_right_link">
-    <inertial>
-      <mass value="1e-5" />
-      <origin xyz="0 0 0" rpy="0 0 0"/>
-      <inertia ixx="1e-6" ixy="0" ixz="0" iyy="1e-6" iyz="0" izz="1e-6" />
-    </inertial>
-  </link>
-  <joint name="zed_camera_left_joint" type="fixed">
-    <origin xyz="0 0.06 0" rpy="0 0 0"/>
-    <parent link="zed_camera_link"/>
-    <child link="camera_link"/>
-    <axis xyz="0 0 1" />
-  </joint>
-  <joint name="zed_camera_right_joint" type="fixed">
-    <origin xyz="0 -0.06 0" rpy="0 0 0"/>
-    <parent link="zed_camera_link"/>
-    <child link="zed_camera_right_link"/>
-    <axis xyz="0 0 1" />
-  </joint>
+  </link>
+  <joint name="left_camera_stereo_joint" type="fixed">
+    <origin xyz="0.0 0 0.0" rpy="0 0 0"/>
+    <parent link="left_camera_link"/>
+    <child link="left_camera_frame"/>
+  </joint>
+  <link name="left_camera_frame"/>
+  <joint name="left_camera_optical_joint" type="fixed">
+    <origin xyz="0.0 0 0.0" rpy="-1.5714 0 -1.5714"/>
+    <parent link="left_camera_frame"/>
+    <child link="left_camera_optical_frame"/>
+  </joint>
+  <link name="left_camera_optical_frame"/>
   <!-- Velodyne URDF, plugin, etc -->
   <xacro:include filename="$(find velodyne_description)/urdf/VLP-16.urdf.xacro"/>

Commit message: Update to the newest version Yuhan

File: src/jackal/jackal_description_rtab/urdf/multi_jackal.urdf.xacro (robot description, xacro)
@@ -237,7 +237,8 @@
   <!-- stereo camera -->
   <joint name="left_camera_joint" type="fixed">
-    <origin xyz="0.7 0 0.3" rpy="0 0 0"/>
-    <parent link="base_link"/>
+    <origin xyz="0.25 0 0.04" rpy="0 0 0"/>
+    <parent link="chassis_link"/>
     <child link="left_camera_link"/>
+    <axis xyz="0 0 1" />
   </joint>
   <link name="left_camera_link">

Commit message: edited gazebo urdf

File: src/jackal/jackal_description_rtab/urdf/multi_jackal.urdf.xacro (robot description, xacro)
@@ -278,5 +278,5 @@
   <xacro:include filename="$(find velodyne_description)/urdf/VLP-16.urdf.xacro"/>
   <VLP-16 parent="front_mount" name="velodyne" topic="/$(arg namespace)/velodyne_points" hz="10" samples="360" gpu="false" lasers="16" max_range="4">
-    <origin xyz="0 0 0.2" rpy="0 0 0" />
+    <origin xyz="0 0 0.05" rpy="0 0 0" />  <!-- og: 0.2 -->
   </VLP-16>
   <link name="land_pad">
@@ -298,5 +298,5 @@
     <parent link="base_link"/>
     <child link="land_pad"/>
-    <origin xyz="0 0 0.38" rpy="0 0 0"/>
+    <origin xyz="0 0 0.21" rpy="0 0 0"/> <!-- og: 0.38 -->
   </joint>
   <!-- Velodyne mount stuff -->
